File: PCB/PCB.kicad_sch (KiCad schematic)
At the start: 10 parts

Commit message: PCB Schematic
Parts:
- removed C?: 1uF, symbol Device:C
- removed J?: XTAL OUT, symbol Connector_Generic:Conn_01x02
- removed J?: 3V SUPPLY, symbol Connector_Generic:Conn_01x02
- removed J?: 1V5 SUPPLY, symbol Connector_Generic:Conn_01x02
- removed R?: 100R, symbol Device:R
- removed R?: 470R, symbol Device:R
- removed U?: MIC5205YM5, Package_TO_SOT_SMD:SOT-23-5, symbol Regulator_Linear:MIC5205YM5
- added C? (x2): 15pF, symbol Device:C
- added C?: 22uF, symbol Device:C
- added C?: 10uF, symbol Device:C
- added D?: BAT54A, Package_TO_SOT_SMD:SOT-23, symbol Diode:BAT54A
- added J?: CLK, symbol Connector_Generic:Conn_01x02
- added J?: BATT, symbol Connector_Generic:Conn_01x02
- added L?: 10uH, symbol Device:L
- added R? (x2): 100R, symbol Device:R
- added R?: 10k, symbol Device:R
- added U?: XC9140MR-G, symbol Custom_IC:XC9140MR-G
- added Y?: 32.768kHz, symbol Device:Crystal
- C?: value 10uF -> 0.1uF
Connections:
- net GND: now also C?.1, C?.1, C?.1, C?.1, D?.3, J?.1 (Pin_1), U?.2 (GND)
- net MISO: now also U?.6 (PB1), R?.1
- net MOSI: now also U?.5 (AREF/PB0), R?.1
- net RST: now also U?.1 (~{RESET}/PB5), R?.2
- net SCK: now also U?.7 (PB2)
- net at U?.2 (XTAL1/PB3): now also C?.2, Y?.2
- net at U?.3 (XTAL2/PB4): now also C?.2, Y?.1
- net +3V0 renamed +3V3
- net +3V3: now also C?.2, R?.1, U?.4 (VOUT)
- new net: D?.2, J?.1 (Pin_1), R?.2
- new net: D?.1, J?.2 (Pin_2), R?.2
- new net: C?.2, J?.2 (Pin_2), L?.1, U?.1 (CE), U?.3 (VBATT)
- new net: L?.2, U?.5 (LX)
Other:
- moved on the sheet: C?
